File: lekirbot PCB/lekirbotv2/lekirbotv2.kicad_pcb (KiCad board)
At the start: 2 copper layers, 104.1 x 155.6 mm, 56 parts, among them IC3 7404D, J1 455-1750-1-ND, J2 455-1750-1-ND, J3 Conn_01x04_Pin, M1A0 CONN_01, M1B0 CONN_01, M2A0 CONN_01, M2B0 CONN_01, SW1 SW_Push, U1 TB6612FNG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

Commit message: Updated lekirbotv2
Parts:
- moved IC3 2.67 mm to (91.6, 133.7), turned to 90 degrees
- moved U1 1.27 mm to (92.0, 133.0), turned to 180 degrees
Routing:
- net +5V: track 0.00 -> 559.1 mm, vias 0 -> 6
- net GND: track 0.00 -> 408.1 mm
- net /IO11: track 0.00 -> 191.9 mm, vias 0 -> 1
- net /IO13: track 0.00 -> 185.3 mm, vias 0 -> 1
- net /AD0: track 0.00 -> 184.3 mm, vias 0 -> 1
- net /AD1: track 0.00 -> 182.3 mm, vias 0 -> 1
- net /AD6: track 0.00 -> 172.7 mm, vias 0 -> 1
- net /IO12: track 0.00 -> 169.0 mm, vias 0 -> 1
- net /IO4: track 0.00 -> 168.5 mm, vias 0 -> 2
- net /IO7: track 0.00 -> 162.4 mm, vias 0 -> 1
- net /AD2: track 0.00 -> 162.2 mm, vias 0 -> 2
- net /AD3: track 0.00 -> 147.4 mm, vias 0 -> 1
- net /AD4: track 0.00 -> 145.7 mm, vias 0 -> 2
- net /AD5: track 0.00 -> 133.1 mm, vias 0 -> 4
- net /IO9: track 0.00 -> 124.8 mm, vias 0 -> 1
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- added copper zone on B.Cu, net GND
- added copper zone on F.Cu, net GND
Other:
- outline, holes or cut-outs redrawn
- board text added: "8 Feb 2024"
- board text added: "LekirBot PCB v2"
- board text removed: "4 Feb 2024"
- board text removed: "LekirBot PCB"
